File: Shield6to_KC4_sin_conectores.kicad_pcb (KiCad board)
At the start: 2 copper layers, 110.5 x 80 mm, 21 parts, among them J1 DB9, P1 CONN_9, P2 CONN_8, P3 CONN_9, P4 CONN_8, P5 CONN_8, P6 CONN_8, P7 CONN_8, P8 CONN_8, U2 MAX232

Commit message: Primera version de la Placa lista para la Revision de MArtín
Parts:
- removed P6, P7: CONN_8, Socket_Strips:Socket_Strip_Straight_1x08
- added D1: LED, LEDs:LED-3MM, F.Cu at (75.6, 131.4)
- added JP3: JUMPER3, Pin_Headers:Pin_Header_Straight_1x03, F.Cu at (111.1, 114.9)
- added R1: R, Resistors_ThroughHole:Resistor_Horizontal_RM10mm, F.Cu at (149.9, 112.4)
- added R2: R, Resistors_ThroughHole:Resistor_Horizontal_RM10mm, F.Cu at (139.7, 114.3)
- added R3: R, Resistors_ThroughHole:Resistor_Horizontal_RM10mm, F.Cu at (137.2, 110.5)
- added R4: R, Resistors_ThroughHole:Resistor_Horizontal_RM10mm, F.Cu at (134.6, 106.7)
- added R5: R, Resistors_ThroughHole:Resistor_Horizontal_RM10mm, F.Cu at (70.5, 123.8)
- added SW1: SW_PUSH, Buttons_Switches_ThroughHole:SW_PUSH_SMALL, F.Cu at (123.2, 125.7)
- added SW2: SW_PUSH, Buttons_Switches_ThroughHole:SW_PUSH_SMALL, F.Cu at (133.3, 125.7)
- added SW3: SW_PUSH, Buttons_Switches_ThroughHole:SW_PUSH_SMALL, F.Cu at (143.5, 125.7)
- added SW4: SW_PUSH, Buttons_Switches_ThroughHole:SW_PUSH_SMALL, F.Cu at (153.7, 125.7)
- added U1: ID-12LA, Librerias:ID12-LA, F.Cu at (68.6, 101.6)
- moved C5 48.5 mm to (113.0, 126.4), turned to 270 degrees
- moved C4 44.4 mm to (105.4, 128.9)
- moved C1 39.9 mm to (88.6, 127.3), turned to 0 degrees
- moved C2 39.8 mm to (96.2, 127.3), turned to 0 degrees
- moved C3 39.5 mm to (111.8, 121.9), turned to 0 degrees
- moved U2 32.9 mm to (88.6, 122.2), turned to 90 degrees
- moved JP2 3.17 mm to (144.8, 65.4)
Connections:
- U2 pad 12: RX -> PC
Routing:
- net +5V: track 219.1 -> 365.5 mm, vias 6 -> 2
- net Tarjeta: track 0.00 -> 56.3 mm, vias 0 -> 2
- net TX: track 57.6 -> 17.2 mm, vias 2 -> 0
- net GND: track 363.0 -> 397.3 mm
- net Net-(J1-Pad2): track 26.2 -> 60.0 mm
- net Net-(R5-Pad2): track 0.00 -> 32.0 mm
- net Net-(J1-Pad3): track 34.4 -> 63.1 mm
- net /RB6: track 21.0 -> 48.5 mm
- net RX: track 52.2 -> 25.3 mm, vias 2 -> 0
- net /RB7: track 21.0 -> 44.9 mm
- net /RD6: track 86.4 -> 65.5 mm
- net /RD5: track 86.3 -> 65.4 mm
- net /RD4: track 86.3 -> 65.4 mm
- net /RD3: track 91.4 -> 70.5 mm
- net /RD2: track 91.0 -> 70.1 mm
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Other:
- board size 110.5 x 80 mm -> 109.2 x 80 mm
- net class Default: via_dia 1.2 -> 1.5
- net class Power: via_dia 1.2 -> 1.5
