File: _autosave-Shield6to_KC4.kicad_pcb (KiCad board)
At the start: 2 copper layers, 110.5 x 80 mm, 21 parts, among them J1 DB9, P1 CONN_9, P2 CONN_8, P3 CONN_9, P4 CONN_8, P5 CONN_8, P6 CONN_8, P7 CONN_8, P8 CONN_8, U2 MAX232

Commit message: Primera version de la Placa lista para la Revision de MArtín
Parts:
- added SW1: SW_PUSH, Buttons_Switches_ThroughHole:SW_PUSH_SMALL, F.Cu at (120.0, 143.5)
- added SW2: SW_PUSH, Buttons_Switches_ThroughHole:SW_PUSH_SMALL, F.Cu at (158.1, 143.5)
- added SW3: SW_PUSH, Buttons_Switches_ThroughHole:SW_PUSH_SMALL, F.Cu at (145.4, 143.5)
- added SW4: SW_PUSH, Buttons_Switches_ThroughHole:SW_PUSH_SMALL, F.Cu at (132.7, 143.5)
- added U1: ID-12LA, Librerias:ID12-LA, F.Cu at (45.7, 116.2)
Other:
- board size 110.5 x 80 mm -> 109.2 x 80 mm
- net class Default: via_dia 1.2 -> 1.5
- net class Power: via_dia 1.2 -> 1.5
