File: _saved_Shield6to_KC4.sch (KiCad schematic (older format))
At the start: 33 parts, among them J1 DB9, P1 CONN_9, P2 CONN_8, P3 CONN_9, P4 CONN_8, P5 CONN_8, P6 CONN_8, P7 CONN_8, P8 CONN_8, SW1 SW_PUSH, SW2 SW_PUSH, SW3 SW_PUSH, SW4 SW_PUSH, U1 ID-12LA, U2 MAX232

Commit message: Primera version de la Placa lista para la Revision de MArtín
Parts:
- JP3: footprint Pin_Headers:Pin_Header_Angled_1x03 -> Pin_Headers:Pin_Header_Straight_1x03
Changed lines of the file:
@@
 F 0 "JP3" V 2050 1851 50  0000 L CNN
 F 1 "JUMPER3" V 2150 1851 50  0000 L CNN
-F 2 "Pin_Headers:Pin_Header_Angled_1x03" H 2100 1750 50  0001 C CNN
+F 2 "Pin_Headers:Pin_Header_Straight_1x03" H 2100 1750 50  0001 C CNN
 F 3 "" H 2100 1750 50  0000 C CNN
 	1    2100 1750
