File: Shield6to_KC4_Con_RFID.kicad_pcb (KiCad board)
At the start: 2 copper layers, 109.2 x 80 mm, 31 parts, among them J1 DB9, P1 CONN_9, P2 CONN_8, P3 CONN_9, P4 CONN_8, P5 CONN_8, P8 CONN_8, SW1 SW_PUSH, SW2 SW_PUSH, SW3 SW_PUSH, SW4 SW_PUSH, U1 ID-12LA, U2 MAX232

Commit message: Changes to be committed: 	renamed:    Librerias.pretty/ID12-LA.kicad_mod -> Modulos/ID12-LA.kicad_mod 	modified:   Shield6to_KC4-cache.lib 	renamed:    _saved_Shield6to_KC4.sch -> Shield6to_KC4.bak 	modified:   Shield6to_KC4.net 	modified:   Shield6to_KC4.sch 	renamed:    Shield6to_KC4_sin_conectores.kicad_pcb -> Shield6to_KC4_Con_RFID.kicad_pcb 	renamed:    Shield6to_KC4.kicad_pcb -> Shield6to_KC4_SinRFID.kicad_pcb 	modified:   Shield6to_KC4_sin_conectores.kicad_pcb-bak 	new file:   Shield6to_KC4_sin_conectores.pro 	deleted:    Shield6to_KICAD4.net 	renamed:    Shield6to_KC4+.kicad_pcb -> _autosave-Shield6to_KC4_sin_conectores.kicad_pcb
Parts:
- added R6: 1K, Resistors_ThroughHole:Resistor_Horizontal_RM10mm, F.Cu at (111.8, 73.7)
- added R7: 10K, Resistors_ThroughHole:Resistor_Horizontal_RM10mm, F.Cu at (108.6, 73.7)
- added SW5: RESET, Buttons_Switches_ThroughHole:SW_PUSH_SMALL, F.Cu at (100.3, 71.8)
- R1, R2, R3, R4: value R -> 10K
- R5: value R -> 3K3
- SW1: value SW_PUSH -> BOOT
- moved SW1 1.91 mm to (123.2, 127.6)
- moved SW2 1.91 mm to (133.3, 127.6)
- moved SW3 1.91 mm to (143.5, 127.6)
- moved SW4 1.91 mm to (153.7, 127.6)
- moved C4 1.27 mm to (105.4, 130.2)
- moved C5 1.27 mm to (113.0, 127.6)
- moved C3 1.27 mm to (111.8, 123.2)
- moved D1 1.27 mm to (75.6, 130.2)
Connections:
- DS1 pad 16: Net-(DS1-Pad16) -> GND
Routing:
- net /RE3: track 4.45 -> 29.8 mm
- net GND: track 397.3 -> 412.8 mm
- net Net-(DS1-Pad15): track 0.00 -> 10.7 mm
- net +5V: track 365.5 -> 370.7 mm
- net /RB7: track 44.9 -> 48.7 mm
- net /RB4: track 36.9 -> 39.6 mm
- net /RD0: track 60.9 -> 63.5 mm
- net /RB6: track 48.5 -> 45.9 mm
- net /RD1: track 68.7 -> 70.9 mm
- net /RB5: track 38.1 -> 40.0 mm
- net Net-(D1-Pad2): track 5.08 -> 3.81 mm
- net Net-(C3-Pad1): track 24.7 -> 26.0 mm
- net Net-(C4-Pad2): track 7.34 -> 7.85 mm
Other:
- board text added: "2015"
- board text added: "EEST1"
- board text added: "R1.0"
- board text added: "Shield 6to"
