File: _autosave-Shield6to_KC4_sin_conectores.kicad_pcb (KiCad board)
At the start: 2 copper layers, 109.2 x 80 mm, 26 parts, among them J1 DB9, P1 CONN_9, P2 CONN_8, P3 CONN_9, P4 CONN_8, P5 CONN_8, P6 CONN_8, P7 CONN_8, P8 CONN_8, SW1 SW_PUSH, SW2 SW_PUSH, SW3 SW_PUSH, SW4 SW_PUSH, U1 ID-12LA, U2 MAX232

Commit message: Changes to be committed: 	renamed:    Librerias.pretty/ID12-LA.kicad_mod -> Modulos/ID12-LA.kicad_mod 	modified:   Shield6to_KC4-cache.lib 	renamed:    _saved_Shield6to_KC4.sch -> Shield6to_KC4.bak 	modified:   Shield6to_KC4.net 	modified:   Shield6to_KC4.sch 	renamed:    Shield6to_KC4_sin_conectores.kicad_pcb -> Shield6to_KC4_Con_RFID.kicad_pcb 	renamed:    Shield6to_KC4.kicad_pcb -> Shield6to_KC4_SinRFID.kicad_pcb 	modified:   Shield6to_KC4_sin_conectores.kicad_pcb-bak 	new file:   Shield6to_KC4_sin_conectores.pro 	deleted:    Shield6to_KICAD4.net 	renamed:    Shield6to_KC4+.kicad_pcb -> _autosave-Shield6to_KC4_sin_conectores.kicad_pcb
Parts:
- removed P6, P7: CONN_8, Socket_Strips:Socket_Strip_Straight_1x08
- added D1: LED, LEDs:LED-3MM, F.Cu at (75.6, 130.2)
- added JP3: JUMPER3, Pin_Headers:Pin_Header_Straight_1x03, F.Cu at (111.1, 114.9)
- added R1: 10K, Resistors_ThroughHole:Resistor_Horizontal_RM10mm, F.Cu at (149.9, 112.4)
- added R2: 10K, Resistors_ThroughHole:Resistor_Horizontal_RM10mm, F.Cu at (139.7, 114.3)
- added R3: 10K, Resistors_ThroughHole:Resistor_Horizontal_RM10mm, F.Cu at (137.2, 110.5)
- added R4: 10K, Resistors_ThroughHole:Resistor_Horizontal_RM10mm, F.Cu at (134.6, 106.7)
- added R5: 3K3, Resistors_ThroughHole:Resistor_Horizontal_RM10mm, F.Cu at (70.5, 123.8)
- added R6: 1K, Resistors_ThroughHole:Resistor_Horizontal_RM10mm, F.Cu at (111.8, 73.7)
- added R7: 10K, Resistors_ThroughHole:Resistor_Horizontal_RM10mm, F.Cu at (108.6, 73.7)
- added SW5: RESET, Buttons_Switches_ThroughHole:SW_PUSH_SMALL, F.Cu at (100.3, 71.8)
- SW1: value SW_PUSH -> BOOT
- moved C5 48.6 mm to (113.0, 127.6), turned to 270 degrees
- moved C4 44.9 mm to (105.4, 130.2)
- moved C1 39.9 mm to (88.6, 127.3), turned to 0 degrees
- moved C2 39.8 mm to (96.2, 127.3), turned to 0 degrees
- moved C3 39.6 mm to (111.8, 123.2), turned to 0 degrees
- moved U2 32.9 mm to (88.6, 122.2), turned to 90 degrees
- moved SW2 29.4 mm to (133.3, 127.6), turned to 180 degrees
- moved U1 27.1 mm to (68.6, 101.6), turned to 90 degrees
- moved SW4 26.3 mm to (153.7, 127.6), turned to 180 degrees
- moved SW1 16.2 mm to (123.2, 127.6), turned to 180 degrees
- moved SW3 16.0 mm to (143.5, 127.6), turned to 180 degrees
- moved JP2 3.17 mm to (144.8, 65.4)
Connections:
- DS1 pad 16: Net-(DS1-Pad16) -> GND
- SW1 pad 1: +5V -> GND
- SW1 pad 2: Net-(R4-Pad2) -> /RB4
- SW2 pad 1: +5V -> GND
- SW2 pad 2: Net-(R3-Pad2) -> /RB5
- SW3 pad 1: +5V -> GND
- SW3 pad 2: Net-(R2-Pad2) -> /RB6
- SW4 pad 1: +5V -> GND
- SW4 pad 2: Net-(R1-Pad2) -> /RB7
- U1 pad 2: Net-(U1-Pad2) -> +5V
- U1 pad 7: Net-(U1-Pad7) -> GND
- U1 pad 8: Net-(U1-Pad8) -> Tarjeta
- U2 pad 12: RX -> PC
Routing:
- net +5V: track 218.9 -> 370.7 mm, vias 6 -> 2
- net Tarjeta: track 0.00 -> 56.3 mm, vias 0 -> 2
- net GND: track 363.0 -> 412.8 mm
- net TX: track 57.6 -> 17.2 mm, vias 2 -> 0
- net Net-(J1-Pad2): track 26.2 -> 60.0 mm
- net Net-(R5-Pad2): track 0.00 -> 32.0 mm
- net Net-(J1-Pad3): track 34.4 -> 63.1 mm
- net /RB7: track 21.0 -> 48.7 mm
- net RX: track 52.2 -> 25.3 mm, vias 2 -> 0
- net /RE3: track 4.45 -> 29.8 mm
- net /RB6: track 21.0 -> 45.9 mm
- net /RD6: track 86.4 -> 65.5 mm
- net /RD5: track 86.3 -> 65.4 mm
- net /RD4: track 86.3 -> 65.4 mm
- net /RD3: track 91.4 -> 70.5 mm
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Other:
- outline, holes or cut-outs redrawn
- board text added: "2015"
- board text added: "EEST1"
- board text added: "R1.0"
- board text added: "Shield 6to"
