File: Shield6to_KC4.kicad_pcb (KiCad board)
At the start: 2 copper layers, 112.4 x 80 mm, 34 parts, among them J1 DB9, P1 CONN_9, P2 CONN_8, P3 CONN_9, P4 CONN_8, P5 CONN_8, P8 CONN_8, SW1 BOOT, SW2 SW_PUSH, SW3 SW_PUSH, SW4 BOT, SW5 RESET, U1 ID-12LA, U2 MAX232

Commit message: modified:   Shield6to_KC4.kicad_pcb 	modified:   Shield6to_KC4.kicad_pcb-bak 	modified:   Shield6to_KC4.net 	new file:   _saved_Shield6to_KC4.sch
Parts:
- removed R5: 3K3, Resistors_ThroughHole:Resistor_Horizontal_RM10mm
- C1, C2: footprint C_Radial_D5_L6_P2.5 -> Capacitors_ThroughHole:C_Radial_D5_L6_P2.5
- J1: footprint DB9FC -> Connect:DB9FC
- SW1: footprint SW_PUSH_SMALL -> Buttons_Switches_ThroughHole:SW_PUSH_SMALL
- moved D1 15.1 mm to (61.6, 124.5), turned to 0 degrees
- turned R6 to 270 degrees
Connections:
- J1 pad : GND -> (no net)
- R6 pad 1: /LED+ -> +5V
- R6 pad 2: +5V -> /LED+
- U1 pad 6: Net-(R5-Pad2) -> Net-(D1-Pad2)
Routing:
- net Net-(R5-Pad2): track 36.5 -> 0.00 mm
- net Net-(D1-Pad2): track 3.81 -> 36.6 mm
- net GND: track 425.6 -> 423.3 mm

Commit message: On branch master  Your branch is up-to-date with 'origin/master'.
 Changes to be committed:
	modified:   Shield6to_KC4.bak
	modified:   Shield6to_KC4.kicad_pcb
	modified:   Shield6to_KC4.kicad_pcb-bak
	modified:   Shield6to_KC4.net
	modified:   Shield6to_KC4.sch
	deleted:    _saved_Shield6to_KC4.sch
Parts:
- moved D1 5.24 mm to (66.7, 125.7), turned to 90 degrees
- moved SW5 0.38 mm to (100.3, 71.4)
Connections:
- P2 pad 3: /RE3 -> /RC2
- P2 pad 4: /RC2 -> /RC1
- P2 pad 5: /RC1 -> /RC0
- P2 pad 6: /RC0 -> /RE3
- P4 pad 3: /RE3 -> /RC2
- P4 pad 4: /RC2 -> /RC1
- P4 pad 5: /RC1 -> /RC0
- P4 pad 6: /RC0 -> /RE3
Routing:
- net GND: track 423.3 -> 403.2 mm, vias 0 -> 2
- net /RE3: track 29.1 -> 28.3 mm

Commit message: Changes to be committed: 	modified:   Shield6to_KC4.kicad_pcb 	modified:   Shield6to_KC4.kicad_pcb-bak
Routing:
- net /RE3: track 28.3 -> 30.4 mm
Other:
- board text added: "R2.1"
- board text removed: "R1.0"
Changed lines of the file:
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@@
   (general
     (links 99)
-    (no_connects 5)
+    (no_connects 0)
     (area 28.195001 33.345 198.5 133.400001)
     (thickness 1.6)
     (drawings 21)
-    (tracks 366)
+    (tracks 367)
     (zones 0)
     (modules 33)
@@
       (net 34 /RB4))
   )
+  (gr_text R2.1 (at 62.103 72.644) (layer B.Cu)
+    (effects (font (size 1.5 1.5) (thickness 0.3)) (justify mirror))
+  )
   (dimension 80.01 (width 0.3) (layer Dwgs.User)
     (gr_text "80,010 mm" (at 34.845 93.345 270) (layer Dwgs.User)
@@
   (gr_line (start 167.64 53.34) (end 55.245 53.34) (layer Edge.Cuts) (width 0.1))
   (gr_line (start 55.245 133.35) (end 167.64 133.35) (layer Edge.Cuts) (width 0.1))
-  (gr_text "R1.0\n" (at 62.23 70.485) (layer B.Cu)
-    (effects (font (size 1.5 1.5) (thickness 0.3)) (justify mirror))
-  )
   (gr_text "Shield\n6to" (at 62.23 87.63) (layer B.Cu)
     (effects (font (size 1.5 1.5) (thickness 0.3)) (justify mirror))
@@
   (segment (start 127 60.96) (end 127 65.405) (width 0.8) (layer B.Cu) (net 41) (status 20))
   (segment (start 124.46 65.405) (end 124.46 60.96) (width 0.8) (layer B.Cu) (net 42) (status 10))
+  (segment (start 104.14 73.914) (end 104.14 77.851) (width 0.8) (layer B.Cu) (net 43))
+  (segment (start 104.14 77.851) (end 105.029 78.74) (width 0.8) (layer B.Cu) (net 43))
+  (segment (start 105.029 78.74) (end 108.585 78.74) (width 0.8) (layer B.Cu) (net 43))
   (segment (start 96.52 73.914) (end 104.14 73.914) (width 0.8) (layer B.Cu) (net 43))
   (segment (start 104.14 73.914) (end 101.6 71.374) (width 0.8) (layer B.Cu) (net 43))
   (segment (start 101.6 71.374) (end 101.6 65.405) (width 0.8) (layer B.Cu) (net 43))
-  (segment (start 108.585 78.74) (end 108.585 78.359) (width 0.8) (layer B.Cu) (net 43))
-  (segment (start 108.585 78.359) (end 104.14 73.914) (width 0.8) (layer B.Cu) (net 43))
   (segment (start 101.6 60.96) (end 101.6 65.405) (width 0.8) (layer B.Cu) (net 43))
   (segment (start 93.98 60.96) (end 93.98 65.405) (width 0.8) (layer B.Cu) (net 44))

Commit message: Changes to be committed: 	new file:   3d_indicators.zip 	new file:   Modelodelgabinete.fcstd 	new file:   Modelodelgabinete.fcstd1 	modified:   Shield6to_KC4.bak 	modified:   Shield6to_KC4.kicad_pcb 	modified:   Shield6to_KC4.kicad_pcb-bak 	modified:   Shield6to_KC4.net 	modified:   Shield6to_KC4.sch 	new file:   box.pro 	new file:   box.stl 	new file:   placaFreeCad.fcstd
Parts:
- SW1: value BOOT -> BOOT/BOT1
- SW2: value SW_PUSH -> BOT2
- SW3: value SW_PUSH -> BOT3
- SW4: value BOT -> BOT4
Routing:
- net Net-(J1-Pad2): track 60.3 -> 45.3 mm
- net Net-(J1-Pad3): track 63.3 -> 48.5 mm
- net GND: track 403.2 -> 391.4 mm
- net /RD1: track 70.9 -> 74.2 mm
- net /RD0: track 63.5 -> 66.4 mm
Changed lines of the file:
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@@
     (thickness 1.6)
     (drawings 21)
-    (tracks 367)
+    (tracks 354)
     (zones 0)
     (modules 33)
@@
       (effects (font (size 1 1) (thickness 0.15)))
     )
-    (fp_text value BOT (at 0 1.016 180) (layer F.Fab)
+    (fp_text value BOT4 (at 0 1.016 180) (layer F.Fab)
       (effects (font (size 1 1) (thickness 0.15)))
     )
@@
       (effects (font (size 1 1) (thickness 0.15)))
     )
-    (fp_text value SW_PUSH (at 0 1.016 180) (layer F.Fab)
+    (fp_text value BOT3 (at 0 1.016 180) (layer F.Fab)
       (effects (font (size 1 1) (thickness 0.15)))
     )
@@
       (effects (font (size 1 1) (thickness 0.15)))
     )
-    (fp_text value SW_PUSH (at 0 1.016 180) (layer F.Fab)
+    (fp_text value BOT2 (at 0 1.016 180) (layer F.Fab)
       (effects (font (size 1 1) (thickness 0.15)))
     )
@@
       (effects (font (size 1 1) (thickness 0.15)))
     )
-    (fp_text value BOOT (at 0 1.016 180) (layer F.Fab)
+    (fp_text value BOOT/BOT1 (at 0 1.016 180) (layer F.Fab)
       (effects (font (size 1 1) (thickness 0.15)))
     )
@@
   (segment (start 106.553 71.12) (end 106.045 71.12) (width 1) (layer B.Cu) (net 5))
   (via (at 106.553 71.12) (size 1.5) (drill 0.7) (layers F.Cu B.Cu) (net 5))
-  (segment (start 97.391787 71.12) (end 106.553 71.12) (width 1) (layer F.Cu) (net 5))
   (via (at 97.391787 71.12) (size 1.5) (drill 0.7) (layers F.Cu B.Cu) (net 5))
-  (segment (start 96.52 68.834) (end 96.52 70.248213) (width 1) (layer B.Cu) (net 5))
-  (segment (start 96.52 70.248213) (end 97.391787 71.12) (width 1) (layer B.Cu) (net 5))
   (segment (start 66.675 125.73) (end 73.279 125.73) (width 1) (layer B.Cu) (net 5))
   (segment (start 73.279 125.73) (end 76.835 122.174) (width 1) (layer B.Cu) (net 5))
@@
   (segment (start 121.92 67.945) (end 122.555 68.58) (width 0.8) (layer B.Cu) (net 10))
   (segment (start 121.92 60.96) (end 121.92 65.405) (width 0.8) (layer B.Cu) (net 10) (status 20))
+  (segment (start 91.44 65.405) (end 91.44 77.851) (width 0.8) (layer B.Cu) (net 11))
+  (segment (start 91.44 77.851) (end 96.139 82.55) (width 0.8) (layer B.Cu) (net 11))
+  (segment (start 96.139 82.55) (end 134.62 82.55) (width 0.8) (layer B.Cu) (net 11))
+  (segment (start 134.62 82.55) (end 135.89 81.28) (width 0.8) (layer B.Cu) (net 11))
+  (segment (start 135.89 81.28) (end 135.89 78.74) (width 0.8) (layer B.Cu) (net 11))
   (segment (start 91.44 65.405) (end 91.44 60.96) (width 0.8) (layer B.Cu) (net 11))
-  (segment (start 91.44 65.405) (end 91.44 73.025) (width 0.8) (layer B.Cu) (net 11) (status 10))
-  (segment (start 135.89 81.28) (end 135.89 78.74) (width 0.8) (layer B.Cu) (net 11) (status 20))
-  (segment (start 134.62 82.55) (end 135.89 81.28) (width 0.8) (layer B.Cu) (net 11))
-  (segment (start 100.965 82.55) (end 134.62 82.55) (width 0.8) (layer B.Cu) (net 11))
-  (segment (start 91.44 73.025) (end 100.965 82.55) (width 0.8) (layer B.Cu) (net 11))
-  (segment (start 138.43 78.74) (end 138.43 82.55) (width 0.8) (layer B.Cu) (net 12) (status 10))
-  (segment (start 88.9 73.025) (end 88.9 65.405) (width 0.8) (layer B.Cu) (net 12) (status 20))
-  (segment (start 100.33 84.455) (end 88.9 73.025) (width 0.8) (layer B.Cu) (net 12))
-  (segment (start 136.525 84.455) (end 100.33 84.455) (width 0.8) (layer B.Cu) (net 12))
+  (segment (start 138.43 78.74) (end 138.43 82.55) (width 0.8) (layer B.Cu) (net 12))
   (segment (start 138.43 82.55) (end 136.525 84.455) (width 0.8) (layer B.Cu) (net 12))
+  (segment (start 136.525 84.455) (end 94.742 84.455) (width 0.8) (layer B.Cu) (net 12))
+  (segment (start 94.742 84.455) (end 88.9 78.613) (width 0.8) (layer B.Cu) (net 12))
+  (segment (start 88.9 78.613) (end 88.9 65.405) (width 0.8) (layer B.Cu) (net 12))
   (segment (start 88.9 65.405) (end 88.9 60.96) (width 0.8) (layer B.Cu) (net 12) (status 10))
   (segment (start 88.9 101.6) (end 88.9 92.075) (width 0.8) (layer B.Cu) (net 13) (status 10))
@@
   (segment (start 107.95 95.885) (end 147.955 95.885) (width 0.8) (layer B.Cu) (net 18))
   (segment (start 106.68 97.155) (end 107.95 95.885) (width 0.8) (layer B.Cu) (net 18))
-  (segment (start 74.93 79.502) (end 75.057 79.375) (width 0.8) (layer B.Cu) (net 20))
-  (segment (start 75.057 79.375) (end 78.105 79.375) (width 0.8) (layer B.Cu) (net 20))
-  (segment (start 83.82 104.775) (end 87.63 108.585) (width 0.8) (layer B.Cu) (net 20))
-  (segment (start 78.105 79.375) (end 81.915 75.565) (width 0.8) (layer B.Cu) (net 20))
-  (segment (start 81.915 75.565) (end 85.09 75.565) (width 0.8) (layer B.Cu) (net 20))
-  (segment (start 87.63 108.585) (end 91.44 108.585) (width 0.8) (layer B.Cu) (net 20))
-  (segment (start 85.09 75.565) (end 88.265 78.74) (width 0.8) (layer B.Cu) (net 20))
-  (segment (start 88.265 78.74) (end 88.265 83.185) (width 0.8) (layer B.Cu) (net 20))
-  (segment (start 88.265 83.185) (end 83.82 87.63) (width 0.8) (layer B.Cu) (net 20))
-  (segment (start 83.82 87.63) (end 83.82 104.775) (width 0.8) (layer B.Cu) (net 20))
-  (segment (start 91.44 108.585) (end 93.6625 110.8075) (width 0.8) (layer B.Cu) (net 20))
-  (segment (start 93.6625 110.8075) (end 93.6625 114.6175) (width 0.8) (layer B.Cu) (net 20))
-  (segment (start 74.93 76.835) (end 77.47 76.835) (width 0.8) (layer B.Cu) (net 21))
-  (segment (start 77.47 76.835) (end 80.645 73.66) (width 0.8) (layer B.Cu) (net 21))
-  (segment (start 86.36 103.505) (end 88.9 106.045) (width 0.8) (layer B.Cu) (net 21))
-  (segment (start 80.645 73.66) (end 86.36 73.66) (width 0.8) (layer B.Cu) (net 21))
-  (segment (start 86.36 73.66) (end 90.805 78.105) (width 0.8) (layer B.Cu) (net 21))
-  (segment (start 88.9 106.045) (end 92.075 106.045) (width 0.8) (layer B.Cu) (net 21))
-  (segment (start 90.805 78.105) (end 90.805 84.455) (width 0.8) (layer B.Cu) (net 21))
-  (segment (start 96.2025 110.1725) (end 96.2025 114.6175) (width 0.8) (layer B.Cu) (net 21))
-  (segment (start 90.805 84.455) (end 86.36 88.9) (width 0.8) (layer B.Cu) (net 21))
-  (segment (start 86.36 88.9) (end 86.36 103.505) (width 0.8) (layer B.Cu) (net 21))
-  (segment (start 92.075 106.045) (end 96.2025 110.1725) (width 0.8) (layer B.Cu) (net 21))
+  (segment (start 93.6625 114.6175) (end 93.6625 110.8075) (width 0.8) (layer B.Cu) (net 20))
+  (segment (start 87.63 108.585) (end 83.82 104.775) (width 0.8) (layer B.Cu) (net 20))
+  (segment (start 93.6625 110.8075) (end 91.44 108.585) (width 0.8) (layer B.Cu) (net 20))
+  (segment (start 91.44 108.585) (end 87.63 108.585) (width 0.8) (layer B.Cu) (net 20))
+  (segment (start 83.82 104.775) (end 83.82 88.011) (width 0.8) (layer B.Cu) (net 20))
+  (segment (start 83.82 88.011) (end 75.311 79.502) (width 0.8) (layer B.Cu) (net 20))
+  (segment (start 75.311 79.502) (end 74.93 79.502) (width 0.8) (layer B.Cu) (net 20))
+  (segment (start 96.2025 114.6175) (end 96.2025 110.1725) (width 0.8) (layer B.Cu) (net 21))
+  (segment (start 96.2025 110.1725) (end 92.075 106.045) (width 0.8) (layer B.Cu) (net 21))
+  (segment (start 88.9 106.045) (end 86.36 103.505) (width 0.8) (layer B.Cu) (net 21))
+  (segment (start 92.075 106.045) (end 88.9 106.045) (width 0.8) (layer B.Cu) (net 21))
+  (segment (start 86.36 103.505) (end 86.36 88.265) (width 0.8) (layer B.Cu) (net 21))
+  (segment (start 86.36 88.265) (end 74.93 76.835) (width 0.8) (layer B.Cu) (net 21))
   (segment (start 160.02 63.881) (end 149.86 63.881) (width 0.8) (layer B.Cu) (net 27))
   (segment (start 149.86 63.881) (end 146.939 60.96) (width 0.8) (layer B.Cu) (net 27))

Commit message: Changes to be committed: 	modified:   Modelodelgabinete.fcstd 	modified:   Modelodelgabinete.fcstd1 	new file:   Modelodelgabinete2.fcstd 	new file:   Modelodelgabinete2.fcstd1 	modified:   Shield6to_KC4.kicad_pcb 	modified:   Shield6to_KC4.kicad_pcb-bak
Routing:
- net GND: vias 2 -> 1
- net (no net): vias 0 -> 1
Changed lines of the file:
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@@
   (general
     (links 99)
-    (no_connects 0)
+    (no_connects 1)
     (area 28.195001 33.345 198.5 133.400001)
     (thickness 1.6)
-    (drawings 21)
+    (drawings 26)
     (tracks 354)
     (zones 0)
@@
     (38 B.Mask user)
     (39 F.Mask user)
-    (40 Dwgs.User user hide)
+    (40 Dwgs.User user)
     (41 Cmts.User user)
     (42 Eco1.User user)
@@
       (effects (font (size 1 1) (thickness 0.15)))
     )
-    (fp_text value JUMPER3 (at 0 -3.1 90) (layer F.Fab)
+    (fp_text value JUMPER3 (at -2.54 2.54 180) (layer F.Fab)
       (effects (font (size 1 1) (thickness 0.15)))
     )
@@
       (net 34 /RB4))
   )
+  (dimension 86.36 (width 0.3) (layer Dwgs.User)
+    (gr_text "86,360 mm" (at 113.03 41.83) (layer Dwgs.User)
+      (effects (font (size 1.5 1.5) (thickness 0.3)))
+    )
+    (feature1 (pts (xy 156.21 57.15) (xy 156.21 40.48)))
+    (feature2 (pts (xy 69.85 57.15) (xy 69.85 40.48)))
+    (crossbar (pts (xy 69.85 43.18) (xy 156.21 43.18)))
+    (arrow1a (pts (xy 156.21 43.18) (xy 155.083496 43.766421)))
+    (arrow1b (pts (xy 156.21 43.18) (xy 155.083496 42.593579)))
+    (arrow2a (pts (xy 69.85 43.18) (xy 70.976504 43.766421)))
+    (arrow2b (pts (xy 69.85 43.18) (xy 70.976504 42.593579)))
+  )
+  (dimension 3.81 (width 0.3) (layer Dwgs.User)
+    (gr_text "3,810 mm" (at 186.135 55.245 90) (layer Dwgs.User)
+      (effects (font (size 1.5 1.5) (thickness 0.3)))
+    )
+    (feature1 (pts (xy 156.21 53.34) (xy 187.485 53.34)))
+    (feature2 (pts (xy 156.21 57.15) (xy 187.485 57.15)))
+    (crossbar (pts (xy 184.785 57.15) (xy 184.785 53.34)))
+    (arrow1a (pts (xy 184.785 53.34) (xy 185.371421 54.466504)))
+    (arrow1b (pts (xy 184.785 53.34) (xy 184.198579 54.466504)))
+    (arrow2a (pts (xy 184.785 57.15) (xy 185.371421 56.023496)))
+    (arrow2b (pts (xy 184.785 57.15) (xy 184.198579 56.023496)))
+  )
+  (dimension 3.81 (width 0.3) (layer Dwgs.User)
+    (gr_text "3,810 mm" (at 43.1 55.245 90) (layer Dwgs.User)
+      (effects (font (size 1.5 1.5) (thickness 0.3)))
+    )
+    (feature1 (pts (xy 69.85 53.34) (xy 41.75 53.34)))
+    (feature2 (pts (xy 69.85 57.15) (xy 41.75 57.15)))
+    (crossbar (pts (xy 44.45 57.15) (xy 44.45 53.34)))
+    (arrow1a (pts (xy 44.45 53.34) (xy 45.036421 54.466504)))
+    (arrow1b (pts (xy 44.45 53.34) (xy 43.863579 54.466504)))
+    (arrow2a (pts (xy 44.45 57.15) (xy 45.036421 56.023496)))
+    (arrow2b (pts (xy 44.45 57.15) (xy 43.863579 56.023496)))
+  )
+  (dimension 11.43 (width 0.3) (layer Dwgs.User)
+    (gr_text "11,430 mm" (at 161.925 45.005) (layer Dwgs.User)
+      (effects (font (size 1.5 1.5) (thickness 0.3)))
+    )
+    (feature1 (pts (xy 156.21 53.34) (xy 156.21 43.655)))
+    (feature2 (pts (xy 167.64 53.34) (xy 167.64 43.655)))
+    (crossbar (pts (xy 167.64 46.355) (xy 156.21 46.355)))
+    (arrow1a (pts (xy 156.21 46.355) (xy 157.336504 45.768579)))
+    (arrow1b (pts (xy 156.21 46.355) (xy 157.336504 46.941421)))
+    (arrow2a (pts (xy 167.64 46.355) (xy 166.513496 45.768579)))
+    (arrow2b (pts (xy 167.64 46.355) (xy 166.513496 46.941421)))
+  )
+  (dimension 14.605 (width 0.3) (layer Dwgs.User)
+    (gr_text "14,605 mm" (at 62.5475 45.005) (layer Dwgs.User)
+      (effects (font (size 1.5 1.5) (thickness 0.3)))
+    )
+    (feature1 (pts (xy 69.85 53.34) (xy 69.85 43.655)))
+    (feature2 (pts (xy 55.245 53.34) (xy 55.245 43.655)))
+    (crossbar (pts (xy 55.245 46.355) (xy 69.85 46.355)))
+    (arrow1a (pts (xy 69.85 46.355) (xy 68.723496 46.941421)))
+    (arrow1b (pts (xy 69.85 46.355) (xy 68.723496 45.768579)))
+    (arrow2a (pts (xy 55.245 46.355) (xy 56.371504 46.941421)))
+    (arrow2b (pts (xy 55.245 46.355) (xy 56.371504 45.768579)))
+  )
+  (dimension 112.395 (width 0.3) (layer Dwgs.User)
+    (gr_text "112,395 mm" (at 111.4425 25.955) (layer Dwgs.User)
+      (effects (font (size 1.5 1.5) (thickness 0.3)))
+    )
+    (feature1 (pts (xy 167.64 53.34) (xy 167.64 24.605)))
+    (feature2 (pts (xy 55.245 53.34) (xy 55.245 24.605)))
+    (crossbar (pts (xy 55.245 27.305) (xy 167.64 27.305)))
+    (arrow1a (pts (xy 167.64 27.305) (xy 166.513496 27.891421)))
+    (arrow1b (pts (xy 167.64 27.305) (xy 166.513496 26.718579)))
+    (arrow2a (pts (xy 55.245 27.305) (xy 56.371504 27.891421)))
+    (arrow2b (pts (xy 55.245 27.305) (xy 56.371504 26.718579)))
+  )
   (gr_text R2.1 (at 62.103 72.644) (layer B.Cu)
     (effects (font (size 1.5 1.5) (thickness 0.3)) (justify mirror))
@@
     (arrow2b (pts (xy 171.45 76.2) (xy 172.036421 77.326504)))
   )
-  (dimension 83.82 (width 0.3) (layer Dwgs.User)
-    (gr_text "83,820 mm" (at 121.92 128.985) (layer Dwgs.User)
-      (effects (font (size 1.5 1.5) (thickness 0.3)))
-    )
-    (feature1 (pts (xy 163.83 120.65) (xy 163.83 130.335)))
-    (feature2 (pts (xy 80.01 120.65) (xy 80.01 130.335)))
-    (crossbar (pts (xy 80.01 127.635) (xy 163.83 127.635)))
-    (arrow1a (pts (xy 163.83 127.635) (xy 162.703496 128.221421)))
-    (arrow1b (pts (xy 163.83 127.635) (xy 162.703496 127.048579)))
-    (arrow2a (pts (xy 80.01 127.635) (xy 81.136504 128.221421)))
-    (arrow2b (pts (xy 80.01 127.635) (xy 81.136504 127.048579)))
-  )
   (dimension 40.64 (width 0.3) (layer Dwgs.User)
     (gr_text "40,640 mm" (at 177.245 81.28 270) (layer Dwgs.User)
@@
   (gr_circle (center 156.21 104.775) (end 157.48 103.505) (layer Edge.Cuts) (width 0.1))
   (gr_circle (center 156.21 57.15) (end 154.94 55.88) (layer Edge.Cuts) (width 0.1))
+  (via (at 97.391787 71.12) (size 1.5) (drill 0.7) (layers F.Cu B.Cu) (net 0))
   (segment (start 88.5825 122.2375) (end 88.5825 127.3175) (width 0.8) (layer B.Cu) (net 1))
   (segment (start 91.0825 127.3175) (end 91.7575 127.3175) (width 0.8) (layer B.Cu) (net 2))
@@
   (segment (start 106.553 71.12) (end 106.045 71.12) (width 1) (layer B.Cu) (net 5))
   (via (at 106.553 71.12) (size 1.5) (drill 0.7) (layers F.Cu B.Cu) (net 5))
-  (via (at 97.391787 71.12) (size 1.5) (drill 0.7) (layers F.Cu B.Cu) (net 5))
   (segment (start 66.675 125.73) (end 73.279 125.73) (width 1) (layer B.Cu) (net 5))
   (segment (start 73.279 125.73) (end 76.835 122.174) (width 1) (layer B.Cu) (net 5))
